Commit message: S

File: omron_app/urdf/system.urdf.xacro (robot description, xacro)
@@ -37,5 +37,5 @@
     <parent link="$(arg prefix)base_link"/>
     <child link="$(arg prefix)base"/>
-    <origin xyz="0.2 -0.0 0.45" rpy=" 0 0 0"/>
+    <origin xyz="0.12 -0.0 0.45" rpy=" 0 0 0"/>
     <axis xyz="0 0 1"/>
   </joint>
